File: MATRIZ 8X8 .brd (EAGLE design)
At the start: 68.6 x 53.3 mm, 137 parts

Commit message: REDISEÑO DE LA MATRIZ SIN TRANSISTORES
REDISEÑO DE LA MATRIZ SIN TRANSISTORES
Parts:
- removed D65, D66: (no value), AUTODESK_CIRCUITS_BREADBOARD:LED5MM
- removed R65, R66, R67, R68, R69, R70, R71, R72, R73: 560‎Ω, AUTODESK_CIRCUITS_BREADBOARD:0207/10
- removed UINTEGRADO FILA 2: (no value), AUTODESK_CIRCUITS_BREADBOARD:DIL16
- removed UINTEGRADO FILA 3: (no value), AUTODESK_CIRCUITS_BREADBOARD:DIL16
- removed UINTEGRADO FILA 4: (no value), AUTODESK_CIRCUITS_BREADBOARD:DIL16
- removed UINTEGRADO FILA 5: (no value), AUTODESK_CIRCUITS_BREADBOARD:DIL16
- removed UINTEGRADO FILA 6: (no value), AUTODESK_CIRCUITS_BREADBOARD:DIL16
- removed UINTEGRADO FILA 7: (no value), AUTODESK_CIRCUITS_BREADBOARD:DIL16
- removed UINTEGRADO FILA 8: (no value), AUTODESK_CIRCUITS_BREADBOARD:DIL16
- removed UINTEGRADO PRIMER FILA: (no value), AUTODESK_CIRCUITS_BREADBOARD:DIL16
- added D1, D2: (no value), AUTODESK_CIRCUITS_BREADBOARD:LED5MM
- added R12, R13, R15, R16, R17, R2, R25, R55, R6: 470‎Ω, AUTODESK_CIRCUITS_BREADBOARD:0207/10
- added U1, U4, U5, U6, U7, U8, U9: (no value), AUTODESK_CIRCUITS_BREADBOARD:DIL16
- added U2: (no value), AUTODESK_CIRCUITS_BREADBOARD:ARDUINO_UNO
- R1, R10, R11, R14, R18, R19, R20, R21, R22, R23, R24, R26, R27, R28, R29, R3, R30, R31, R32, R33, R34, R35, R36, R37, R38, R39, R4, R40, R41, R42, R43, R44, R45, R46, R47, R48, R49, R5, R50, R51, R52, R53, R54, R56, R57, R58, R59, R60, R61, R62, R63, R64, R7, R8, R9: value 560‎Ω -> 470‎Ω
- U3: device AUTODESK_CIRCUITS_BREADBOARD:ARDUINO_UNO -> AUTODESK_CIRCUITS_BREADBOARD:DIL16
- moved R14 889.0 mm to (5.00, 1102.3)
- moved U3 838.2 mm to (5.00, 848.3)
- moved R35 838.2 mm to (5.00, 1369.0)
- moved R42 812.8 mm to (5.00, 1457.9)
- moved R49 787.4 mm to (5.00, 1546.8)
- moved R56 762.0 mm to (5.00, 1635.7)
- moved D63 698.5 mm to (5.00, 721.3)
- moved D16 533.4 mm to (5.00, 734.0)
- moved D24 431.8 mm to (5.00, 746.7)
- moved R28 355.6 mm to (5.00, 1280.1)
- moved D32 342.9 mm to (5.00, 759.4)
- moved D40 254.0 mm to (5.00, 772.1)
- moved D48 152.4 mm to (5.00, 784.8)
- moved D57 127.0 mm to (5.00, 645.1)
- moved D58 127.0 mm to (5.00, 657.8)
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Connections:
- net N$1: now also R25.1, U5.15; no longer D25.A, R1.1
- net N$10: now also U1.11, U2.4, U3.11, U4.11, U5.11, U6.11, U7.11, U8.11, U9.11; no longer D6.A, R5.2
- net N$100: now also R47.1, U8.6; no longer R39.2, UINTEGRADO FILA 4.3
- net N$101: now also R48.1, U8.7; no longer R38.2, UINTEGRADO FILA 4.4
- net N$102: now also D47.A, R48.2; no longer R37.2, UINTEGRADO FILA 4.5
- net N$103: now also U7.14, U8.9; no longer R36.2, UINTEGRADO FILA 4.6
- net N$104: now also D51.A, R51.2; no longer R34.2, UINTEGRADO FILA 4.7
- net N$105: now also R50.1, U7.1; no longer R35.2, UINTEGRADO FILA 5.15
- net N$106: now also D50.A, R50.2; no longer R43.2, UINTEGRADO FILA 5.1
- net N$107: now also R49.1, U7.15; no longer R44.2, UINTEGRADO FILA 5.2
- net N$108: now also R51.1, U7.2; no longer R45.2, UINTEGRADO FILA 5.3
- net N$109: now also R52.1, U7.3; no longer R46.2, UINTEGRADO FILA 5.4
- net N$11: now also R30.1, U5.5; no longer D5.A, R8.2
- net N$110: now also D53.A, R52.2; no longer R47.2, UINTEGRADO FILA 5.5
- net N$111: now also R53.1, U7.4; no longer R48.2, UINTEGRADO FILA 5.6
- net N$112: now also D54.A, R53.2; no longer R50.2, UINTEGRADO FILA 5.7
- net N$113: now also R54.1, U7.5; no longer R42.2, UINTEGRADO FILA 6.15
- net N$114: now also D52.A, R54.2; no longer R59.2, UINTEGRADO FILA 6.1
- net N$115: now also D55.A, R55.2; no longer R58.2, UINTEGRADO FILA 6.2
- net N$116: now also R55.1, U7.6; no longer R57.2, UINTEGRADO FILA 6.3
- net N$117: now also R56.1, U7.7; no longer R54.2, UINTEGRADO FILA 6.4
- net N$118: now also D56.A, R56.2; no longer R53.2, UINTEGRADO FILA 6.5
- net N$119: now also U6.14, U7.9; no longer R52.2, UINTEGRADO FILA 6.6
- net N$12: now also R1.1, U1.15; no longer D4.A, R9.2
- net N$120: now also D58.A, R59.2; no longer R51.2, UINTEGRADO FILA 6.7
- net N$121: now also R58.1, U6.1; no longer R49.2, UINTEGRADO FILA 7.15
- net N$122: now also D64.A, R58.2; no longer R66.2, UINTEGRADO FILA 7.1
- net N$123: now also R57.1, U6.15; no longer R65.2, UINTEGRADO FILA 7.2
- net N$124: now also R59.1, U6.2; no longer R64.2, UINTEGRADO FILA 7.3
- net N$125: now also R60.1, U6.3; no longer R63.2, UINTEGRADO FILA 7.4
- net N$126: now also D59.A, R60.2; no longer R62.2, UINTEGRADO FILA 7.5
- net N$127: now also R61.1, U6.4; no longer R61.2, UINTEGRADO FILA 7.6
- net N$128: now also D60.A, R61.2; no longer R60.2, UINTEGRADO FILA 7.7
- net N$129: now also R62.1, U6.5; no longer R56.2, UINTEGRADO FILA 8.15
- net N$13: now also U1.10, U1.16, U2.5V, U3.10, U3.16, U4.10, U4.16, U5.10, U5.16, U6.10, U6.16, U7.10, U7.16, U8.10, U8.16, U9.10, U9.16; no longer D3.A, R10.2
- net N$130: now also D61.A, R62.2; no longer R73.2, UINTEGRADO FILA 8.1
- net N$131: now also D62.A, R63.2; no longer R72.2, UINTEGRADO FILA 8.2
- net N$132: now also R63.1, U6.6; no longer R71.2, UINTEGRADO FILA 8.3
- net N$133: now also R64.1, U6.7; no longer R70.2, UINTEGRADO FILA 8.4
- net N$134: now also R33.1, U9.15; no longer R69.2, UINTEGRADO FILA 8.5
- net N$135: now also R34.1, U9.1; no longer R68.2, UINTEGRADO FILA 8.6
- net N$136: now also U1.9, U3.14; no longer R67.2, UINTEGRADO FILA 8.7
- net N$137: now also U3.9, U4.14; no longer U3.5, UINTEGRADO FILA 2.11, UINTEGRADO FILA 3.11, UINTEGRADO FILA 4.11, UINTEGRADO FILA 5.11, UINTEGRADO FILA 6.11, UINTEGRADO FILA 7.11, UINTEGRADO FILA 8.11, UINTEGRADO PRIMER FILA.11
- net N$138: now also D63.A, R64.2; no longer U3.4, UINTEGRADO FILA 2.12, UINTEGRADO FILA 3.12, UINTEGRADO FILA 4.12, UINTEGRADO FILA 5.12, UINTEGRADO FILA 6.12, UINTEGRADO FILA 7.12, UINTEGRADO FILA 8.12, UINTEGRADO PRIMER FILA.12
- net N$139: now also D1.K, D10.K, D11.K, D12.K, D13.K, D14.K, D15.K, D16.K, D17.K, D18.K, D19.K, D2.K, D20.K, D21.K, D22.K, D23.K, D24.K, D25.K, D26.K, D27.K, D28.K, D29.K, D3.K, D30.K, D31.K, D32.K, D33.K, D34.K, D35.K, D36.K, D37.K, D38.K, D39.K, D4.K, D40.K, D41.K, D42.K, D43.K, D44.K, D45.K, D46.K, D47.K, D48.K, D49.K, D5.K, D50.K, D51.K, D52.K, D53.K, D54.K, D55.K, D56.K, D57.K, D58.K, D59.K, D6.K, D60.K, D61.K, D62.K, D63.K, D64.K, D7.K, D8.K, D9.K, U1.13, U1.8, U2.GND.., U3.13, U3.8, U4.13, U4.8, U5.13, U5.8, U6.13, U6.8, U7.13, U7.8, U8.13, U8.8, U9.13, U9.8; no longer U3.2, UINTEGRADO PRIMER FILA.14
- net N$14: now also D26.A, R34.2; no longer D63.A, R11.2
- net N$140: now also U5.9, U9.14; no longer U3.5V, UINTEGRADO FILA 2.10, UINTEGRADO FILA 2.16, UINTEGRADO FILA 3.10, UINTEGRADO FILA 3.16, UINTEGRADO FILA 4.10, UINTEGRADO FILA 4.16, UINTEGRADO FILA 5.10, UINTEGRADO FILA 5.16, UINTEGRADO FILA 6.10, UINTEGRADO FILA 6.16, UINTEGRADO FILA 7.10, UINTEGRADO FILA 7.16, UINTEGRADO FILA 8.10, UINTEGRADO FILA 8.16, UINTEGRADO PRIMER FILA.10, UINTEGRADO PRIMER FILA.16
- net N$15: now also D27.A, R36.2; no longer D10.K, D11.K, D12.K, D13.K, D14.K, D15.K, D16.K, D17.K, D18.K, D19.K, D20.K, D21.K, D22.K, D23.K, D24.K, D25.K, D26.K, D27.K, D28.K, D29.K, D3.K, D30.K, D31.K, D32.K, D33.K, D34.K, D35.K, D36.K, D37.K, D38.K, D39.K, D4.K, D40.K, D41.K, D42.K, D43.K, D44.K, D45.K, D46.K, D47.K, D48.K, D49.K, D5.K, D50.K, D51.K, D52.K, D53.K, D54.K, D55.K, D56.K, D57.K, D58.K, D59.K, D6.K, D60.K, D61.K, D62.K, D63.K, D64.K, D65.K, D66.K, D7.K, D8.K, D9.K, U3.GND., UINTEGRADO FILA 2.13, UINTEGRADO FILA 2.8, UINTEGRADO FILA 3.13, UINTEGRADO FILA 3.8, UINTEGRADO FILA 4.13, UINTEGRADO FILA 4.8, UINTEGRADO FILA 5.13, UINTEGRADO FILA 5.8, UINTEGRADO FILA 6.13, UINTEGRADO FILA 6.8, UINTEGRADO FILA 7.13, UINTEGRADO FILA 7.8, UINTEGRADO FILA 8.13, UINTEGRADO FILA 8.8, UINTEGRADO PRIMER FILA.13, UINTEGRADO PRIMER FILA.8
- net N$16: now also D3.A, R3.2; no longer D17.A, R14.1
- net N$17: now also R3.1, U1.2; no longer D16.A, R18.1
- net N$18: now also U1.14, U2.2; no longer D15.A, R19.1
- net N$19: now also D4.A, R4.2; no longer D14.A, R20.1
- net N$2: now also R4.1, U1.3; no longer D33.A, R28.1
- net N$20: now also D5.A, R5.2; no longer D13.A, R21.1
- net N$21: now also R5.1, U1.4; no longer D12.A, R22.1
- net N$22: now also D6.A, R6.2; no longer D11.A, R23.1
- net N$23: now also R6.1, U1.5; no longer D10.A, R24.1
- net N$24: now also D7.A, R7.2; no longer D24.A, R26.1
- net N$25: now also R7.1, U1.6; no longer D23.A, R27.1
- net N$26: now also D8.A, R8.2; no longer D22.A, R29.1
- net N$27: now also R8.1, U1.7; no longer D21.A, R30.1
- net N$28: now also D35.A, R12.2; no longer D20.A, R31.1
- net N$29: now also D40.A, R11.2; no longer D19.A, R32.1
- net N$3: now also R20.1, U4.3; no longer D41.A, R35.1
- net N$30: now also D34.A, R10.2; no longer D18.A, R33.1
- net N$31: now also R10.1, U3.1; no longer D26.A, R34.1
- net N$32: now also R9.1, U3.15; no longer D27.A, R36.1
- net N$33: now also R11.1, U3.2; no longer D28.A, R37.1
- net N$34: now also R12.1, U3.3; no longer D29.A, R38.1
- net N$35: now also D36.A, R13.2; no longer D30.A, R39.1
- net N$36: now also R13.1, U3.4; no longer D31.A, R40.1
- net N$37: now also D37.A, R14.2; no longer D32.A, R41.1
- net N$38: now also R14.1, U3.5; no longer D40.A, R43.1
- net N$39: now also D38.A, R15.2; no longer D39.A, R44.1
- net N$4: now also D33.A, R9.2; no longer D49.A, R42.1
- net N$40: now also R15.1, U3.6; no longer D38.A, R45.1
- net N$41: now also D39.A, R16.2; no longer D37.A, R46.1
- net N$42: now also R16.1, U3.7; no longer D36.A, R47.1
- net N$43: now also D19.A, R28.2; no longer D35.A, R48.1
- net N$44: now also D16.A, R19.2; no longer D34.A, R50.1
- net N$45: now also D10.A, R18.2; no longer D42.A, R51.1
- net N$46: now also R18.1, U4.1; no longer D43.A, R52.1
- net N$47: now also R17.1, U4.15; no longer D44.A, R53.1
- net N$48: now also R19.1, U4.2; no longer D45.A, R54.1
- net N$49: now also D11.A, R20.2; no longer D46.A, R57.1
- net N$5: now also D9.A, R17.2; no longer D57.A, R49.1
- net N$50: now also R21.1, U4.4; no longer D47.A, R58.1
- net N$51: now also D12.A, R21.2; no longer D48.A, R59.1
- net N$52: now also D14.A, R22.2; no longer D50.A, R60.1
- net N$53: now also R22.1, U4.5; no longer D51.A, R61.1
- net N$54: now also D15.A, R23.2; no longer D52.A, R62.1
- net N$55: now also R23.1, U4.6; no longer D53.A, R63.1
- net N$56: now also D13.A, R24.2; no longer D54.A, R64.1
- net N$57: now also R24.1, U4.7; no longer D55.A, R65.1
- net N$58: now also D17.A, R25.2; no longer D56.A, R66.1
- net N$59: now also D24.A, R26.2; no longer D58.A, R67.1
- net N$6: now also D25.A, R33.2; no longer D66.A, R56.1
- net N$60: now also R26.1, U5.1; no longer D59.A, R68.1
- net N$61: now also D18.A, R27.2; no longer D60.A, R69.1
- net N$62: now also R27.1, U5.2; no longer D61.A, R70.1
- net N$63: now also U4.9, U5.14; no longer D62.A, R71.1
- net N$64: now also R28.1, U5.3; no longer D64.A, R72.1
- net N$65: now also R29.1, U5.4; no longer D65.A, R73.1
- net N$66: now also D20.A, R29.2; no longer R7.2, UINTEGRADO PRIMER FILA.15
- net N$67: now also U1.12, U2.3, U3.12, U4.12, U5.12, U6.12, U7.12, U8.12, U9.12; no longer R3.2, UINTEGRADO PRIMER FILA.1
- net N$68: now also D21.A, R30.2; no longer R4.1, UINTEGRADO PRIMER FILA.2
- net N$69: now also D22.A, R31.2; no longer R5.1, UINTEGRADO PRIMER FILA.3
- net N$7: now also D41.A, R41.2; no longer D9.A, R7.1
- net N$70: now also R31.1, U5.6; no longer R8.1, UINTEGRADO PRIMER FILA.4
- net N$71: now also D23.A, R32.2; no longer R9.1, UINTEGRADO PRIMER FILA.5
- net N$72: now also R32.1, U5.7; no longer R10.1, UINTEGRADO PRIMER FILA.6
- net N$73: now also D1.A, R2.2; no longer R11.1, UINTEGRADO PRIMER FILA.7
- net N$74: now also D2.A, R1.2; no longer UINTEGRADO FILA 2.14, UINTEGRADO PRIMER FILA.9
- net N$75: now also R2.1, U1.1; no longer UINTEGRADO FILA 3.9, UINTEGRADO FILA 4.14
- net N$76: now also D32.A, R35.2; no longer UINTEGRADO FILA 4.9, UINTEGRADO FILA 5.14
- net N$77: now also R35.1, U9.2; no longer UINTEGRADO FILA 5.9, UINTEGRADO FILA 6.14
- net N$78: now also R36.1, U9.3; no longer UINTEGRADO FILA 6.9, UINTEGRADO FILA 7.14
- net N$79: now also R37.1, U9.4; no longer UINTEGRADO FILA 7.9, UINTEGRADO FILA 8.14
- net N$8: now also D49.A, R49.2; no longer D8.A, R3.1
- net N$80: now also D28.A, R37.2; no longer UINTEGRADO FILA 2.9, UINTEGRADO FILA 3.14
- net N$81: now also R38.1, U9.5; no longer R14.2, UINTEGRADO FILA 2.15
- net N$82: now also D29.A, R38.2; no longer R18.2, UINTEGRADO FILA 2.1
- net N$83: now also D30.A, R39.2; no longer R19.2, UINTEGRADO FILA 2.2
- net N$84: now also R39.1, U9.6; no longer R20.2, UINTEGRADO FILA 2.3
- net N$85: now also R40.1, U9.7; no longer R21.2, UINTEGRADO FILA 2.4
- net N$86: now also D31.A, R40.2; no longer R22.2, UINTEGRADO FILA 2.5
- net N$87: now also U8.14, U9.9; no longer R23.2, UINTEGRADO FILA 2.6
- net N$88: now also D43.A, R43.2; no longer R24.2, UINTEGRADO FILA 2.7
- net N$89: now also R42.1, U8.1; no longer R1.2, UINTEGRADO FILA 3.15
- net N$9: now also D57.A, R57.2; no longer D7.A, R4.2
- net N$90: now also D42.A, R42.2; no longer R26.2, UINTEGRADO FILA 3.1
- net N$91: now also R41.1, U8.15; no longer R27.2, UINTEGRADO FILA 3.2
- net N$92: now also R43.1, U8.2; no longer R29.2, UINTEGRADO FILA 3.3
- net N$93: now also R44.1, U8.3; no longer R30.2, UINTEGRADO FILA 3.4
- net N$94: now also D45.A, R44.2; no longer R31.2, UINTEGRADO FILA 3.5
- net N$95: now also R45.1, U8.4; no longer R32.2, UINTEGRADO FILA 3.6
- net N$96: now also D46.A, R45.2; no longer R33.2, UINTEGRADO FILA 3.7
- net N$97: now also R46.1, U8.5; no longer R28.2, UINTEGRADO FILA 4.15
- net N$98: now also D44.A, R46.2; no longer R41.2, UINTEGRADO FILA 4.1
- net N$99: now also D48.A, R47.2; no longer R40.2, UINTEGRADO FILA 4.2
